File: Led-Controller.kicad_sch (KiCad schematic)
At the start: 62 parts, among them J1 Barrel_Jack, J2 Screw_Terminal, J3 Program, Q1 CSD18540Q5B, Q2 CSD18540Q5B, Q3 CSD18540Q5B, Q4 CSD18540Q5B, Q5 CSD18540Q5B, Q6 CSD18540Q5B, U1 1ED44175N01BXTSA1, U2 1ED44175N01BXTSA1, U3 TPS5430DDA, U4 1ED44175N01BXTSA1, U5 1ED44175N01BXTSA1, U6 TPS5430DDA, U7 1ED44175N01BXTSA1, U8 ESP32-WROOM-32E

Commit message: Final Layout of alpha version 2 (#24)
* Did basic routing for voltage regulators

* Final Layout of PCB version 2 alpha
Parts:
- removed C8: 22uf, Capacitor_SMD:C_0805_2012Metric, symbol Device:C_Small
- added TP1, TP2, TP3, TP4, TP5, TP6, TP7: ~, TestPoint:TestPoint_Pad_D1.0mm, symbol Connector:TestPoint
- C1: renamed from C22; Package (none) -> 402
- C10: renamed from C15; Package (none) -> 805
- C11: renamed from C2; Package (none) -> 402
- C12: renamed from C9; Package (none) -> 402
- C13: renamed from C16; Package (none) -> 402
- C14: renamed from C17; footprint Capacitor_SMD:C_0805_2012Metric_Pad1.18x1.45mm_HandSolder -> Capacitor_SMD:C_0805_2012Metric; Package (none) -> 805
- C15: renamed from C18; footprint Capacitor_SMD:C_0805_2012Metric_Pad1.18x1.45mm_HandSolder -> Capacitor_SMD:C_0805_2012Metric; Package (none) -> 805
- C16: renamed from C19; footprint Capacitor_SMD:C_0805_2012Metric_Pad1.18x1.45mm_HandSolder -> Capacitor_SMD:C_0805_2012Metric; Package (none) -> 805
- C17: renamed from C3; Package (none) -> 402
- C18: renamed from C10; Package (none) -> 402
- C19: renamed from C20; footprint Capacitor_SMD:C_0805_2012Metric_Pad1.18x1.45mm_HandSolder -> Capacitor_SMD:C_0805_2012Metric; Package (none) -> 805
- C2: renamed from C1; footprint Capacitor_SMD:C_0805_2012Metric_Pad1.18x1.45mm_HandSolder -> Capacitor_SMD:C_0805_2012Metric; Package (none) -> 805
- C20: renamed from C21; footprint Capacitor_SMD:C_0805_2012Metric_Pad1.18x1.45mm_HandSolder -> Capacitor_SMD:C_0805_2012Metric; Package (none) -> 805
- C3: renamed from C6; footprint Capacitor_SMD:C_0805_2012Metric_Pad1.18x1.45mm_HandSolder -> Capacitor_SMD:C_0805_2012Metric; Package (none) -> 805
- C4: renamed from C13; footprint Capacitor_SMD:C_0805_2012Metric_Pad1.18x1.45mm_HandSolder -> Capacitor_SMD:C_0805_2012Metric; Package (none) -> 805
- C5: renamed from C23; Package (none) -> 402
- C6: renamed from C4; Package (none) -> 402
- C7: renamed from C11; Package (none) -> 402
- C8: renamed from C14; Package (none) -> 805
- C9: renamed from C7; Package (none) -> 805
- D1: renamed from D2; Package (none) -> SOD-123
- D2: renamed from D3; Package (none) -> SOD-123
- FB1: renamed from FB2; Package (none) -> 805
- FB2: renamed from FB1; Package (none) -> 805
- Q1, Q2: Package (none) -> TDSON 8
- Q3: renamed from Q4; Package (none) -> TDSON 8
- Q4: renamed from Q6; Package (none) -> TDSON 8
- Q5: renamed from Q3; Package (none) -> TDSON 8
- Q6: renamed from Q5; Package (none) -> TDSON 8
- R1: renamed from R17; MANUFACTURER (none) -> Any; Package (none) -> 402
- R10: renamed from R14; MANUFACTURER (none) -> Any; Package (none) -> 402
- R11: renamed from R2; MANUFACTURER (none) -> Any; Package (none) -> 402
- R12: renamed from R7; MANUFACTURER (none) -> Any; Package (none) -> 402
- R13: renamed from R12; MANUFACTURER (none) -> Any; Package (none) -> 402
- R14: renamed from R5; MANUFACTURER (none) -> Any; Package (none) -> 402
- R15: renamed from R11; MANUFACTURER (none) -> Any; Package (none) -> 402
- R16: renamed from R3; MANUFACTURER (none) -> Any; Package (none) -> 402
- R17: renamed from R8; MANUFACTURER (none) -> Any; Package (none) -> 402
- R2: renamed from R1; MANUFACTURER (none) -> Any; Package (none) -> 402
- R3: renamed from R6; MANUFACTURER (none) -> Any; Package (none) -> 402
- R4: renamed from R9; MANUFACTURER (none) -> Any; Package (none) -> 402
- R5: renamed from R13; MANUFACTURER (none) -> Any; Package (none) -> 402
- R6: renamed from R15; MANUFACTURER (none) -> Any; Package (none) -> 402
- R7: renamed from R16; MANUFACTURER (none) -> Any; Package (none) -> 402
- R8: renamed from R4; MANUFACTURER (none) -> Any; Package (none) -> 402
- R9: renamed from R10; MANUFACTURER (none) -> Any; Package (none) -> 402
- U1: renamed from U3; MANUFACTURER (none) -> Texas Instrument; Package (none) -> SOIC 8
- U2: renamed from U6; MANUFACTURER (none) -> Texas Instrument; Package (none) -> SOIC 8
- U3: renamed from U8; MANUFACTURER (none) -> Espresiff
- renumbered D1 to D3, J3 to J1, J1 to J2, J2 to J3, U1 to U4, U4 to U5, U7 to U6, U2 to U7, U5 to U8
Connections:
- net +3.3V: now also TP2.1
- net +9V: now also TP1.1
- net IN1: now also U3.8 (IO32), TP6.1; no longer U3.12 (IO27)
- net IN2: now also U3.9 (IO33), TP7.1; no longer U3.11 (IO26)
- net IN3: now also TP3.1
- net IN4: now also U3.11 (IO26), TP4.1; no longer U3.9 (IO33)
- net IN5: now also U3.12 (IO27), TP5.1; no longer U3.8 (IO32)
Other:
- moved on the sheet: C5, C9, R1, U3
